File: JP65.kicad_pcb (KiCad board)
At the start: 2 copper layers, 285 x 95.1 mm, 153 parts, among them SW1 SW_Push, U1 ATmega32U4-MU, U2 PRTR5V0U2X, Y1 16MHz

Commit message: Make PCB
Parts:
- removed K_RALT1, K_RGUI1: MX-NoLED, MX_Only:MXOnly-1U-Hotswap
- removed K_SRSFT2: MX-NoLED, MX_Only:MXOnly-1.75U-Hotswap
- removed the REF** at (267.5, 219.9)
- added D37: SOD-123, Diode_SMD:D_SOD-123, B.Cu at (408.8, 183.4)
- added D43: SOD-123, Diode_SMD:D_SOD-123, B.Cu at (412.0, 203.2)
- added D48: SOD-123, Diode_SMD:D_SOD-123, B.Cu at (412.0, 222.2)
- added D53: SOD-123, Diode_SMD:D_SOD-123, B.Cu at (412.0, 241.3)
- added D58: SOD-123, Diode_SMD:D_SOD-123, B.Cu at (406.4, 254.0)
- added K_DOWN1: MX-NoLED, MX_Only:MXOnly-1U-Hotswap, F.Cu at (400.8, 258.0)
- added K_EX1: MX-NoLED, MX_Only:MXOnly-1U-Hotswap, F.Cu at (419.9, 181.8)
- added K_EX2: MX-NoLED, MX_Only:MXOnly-1U-Hotswap, F.Cu at (419.9, 200.8)
- added K_EX3: MX-NoLED, MX_Only:MXOnly-1U-Hotswap, F.Cu at (419.9, 219.9)
- added K_EX4: MX-NoLED, MX_Only:MXOnly-1U-Hotswap, F.Cu at (419.9, 238.9)
- added K_LEFT1: MX-NoLED, MX_Only:MXOnly-1U-Hotswap, F.Cu at (381.8, 258.0)
- added K_RIGHT1: MX-NoLED, MX_Only:MXOnly-1U-Hotswap, F.Cu at (419.9, 258.0)
- added K_UP1: MX-NoLED, MX_Only:MXOnly-1U-Hotswap, F.Cu at (400.8, 238.9)
- added REF**: 65, locallib:65_Modded, F.Cu at (77.0, 124.6)
- K_RSFT1: renamed from K_SRSFT1; footprint MX_Only:MXOnly-1U-Hotswap -> MX_Only:MXOnly-1.75U-Hotswap
- moved K_RCTRL1 38.1 mm to (360.4, 258.0)
- moved D67 30.2 mm to (408.8, 241.3)
- moved D74 22.1 mm to (409.6, 254.0)
- moved D1 18.3 mm to (188.1, 259.6)
- moved D27 13.5 mm to (371.5, 259.6)
- moved D22 7.14 mm to (382.6, 240.5)
- moved K_RSFT1 7.14 mm to (374.6, 238.9)
- moved D63 2.38 mm to (368.3, 259.6)
- moved D11 2.38 mm to (168.3, 259.6)
- moved G*** 0.79 mm to (296.1, 258.0)
- turned K_LGUI1 to 180 degrees
- turned K_NFER1 to 90 degrees
Connections:
- K_LGUI1 pad 1: COL1 -> Net-(D11-Pad2)
- K_LGUI1 pad 2: Net-(D11-Pad2) -> COL1
- K_RCTRL1 pad 1: COL13 -> COL11
- K_RCTRL1 pad 2: Net-(D74-Pad2) -> Net-(D63-Pad2)
- U1 pad 10: Net-(U1-Pad10) -> COL14
Routing:
- net COL14: track 0.00 -> 295.1 mm, vias 0 -> 8
- net ROW4: track 328.0 -> 384.0 mm
- net ROW1: track 290.0 -> 325.8 mm
- net ROW3: track 207.0 -> 240.7 mm
- net ROW2: track 315.3 -> 344.3 mm
- net Net-(D37-Pad2): track 0.00 -> 25.7 mm
- net Net-(D67-Pad2): track 29.8 -> 6.68 mm
- net Net-(D53-Pad2): track 0.00 -> 22.3 mm
- net Net-(D43-Pad2): track 0.00 -> 22.3 mm
- net Net-(D48-Pad2): track 0.00 -> 22.2 mm
- net Net-(D58-Pad2): track 0.00 -> 20.9 mm
- net ROW0: track 309.3 -> 329.3 mm
- net Net-(D27-Pad2): track 5.89 -> 21.7 mm
- net COL3: track 142.0 -> 157.5 mm
- net Net-(D74-Pad2): track 25.0 -> 9.97 mm
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Other:
- board size 285 x 95.1 mm -> 303.2 x 94.5 mm
- board text added: "JP65"
- board text added: "JP65 R1.0 20210717 ai03.com"
- board text removed: "JP60"
- board text removed: "JP60 R1.0 20210717 | ai03.com"
