File: JP65.sch (KiCad schematic (older format))
At the start: 21 parts, among them SW1 SW_Push, U1 ATmega32U4-MU, U2 PRTR5V0U2X, Y1 16MHz

Commit message: Make PCB
Connections:
- net COL14: now reaches U1.10 (PB2)
Changed lines of the file:
@@
 EESchema Schematic File Version 4
-LIBS:JIS60-cache
+LIBS:JP65-cache
 EELAYER 30 0
 EELAYER END
@@
 Text GLabel 3000 4800 2    60   Input ~ 0
 COL6
+Text GLabel 3000 4100 2    50   Input ~ 0
+COL14
 $EndSCHEMATC
