File: matrix.sch (KiCad schematic (older format))
At the start: 129 parts

Commit message: Make PCB
Parts:
- added D37, D43, D48, D53, D58: SOD-123, Diode_SMD:D_SOD-123, symbol Device:D_Small
- added K_EX1, K_EX2, K_EX3, K_EX4, K_RIGHT1: MX-NoLED, MX_Only:MXOnly-1U-Hotswap, symbol MX_Alps_Hybrid:MX-NoLED
- K_DOWN1: renamed from K_RCTRL1; footprint MX_Only:MXOnly-1.25U-Hotswap -> MX_Only:MXOnly-1U-Hotswap
- K_RCTRL1: renamed from K_RALT1; footprint MX_Only:MXOnly-1U-Hotswap -> MX_Only:MXOnly-1.25U-Hotswap
- K_RSFT1: renamed from K_SRSFT1; footprint MX_Only:MXOnly-1U-Hotswap -> MX_Only:MXOnly-1.75U-Hotswap
- K_UP1: renamed from K_SRSFT2; footprint MX_Only:MXOnly-1.75U-Hotswap -> MX_Only:MXOnly-1U-Hotswap
- renumbered K_RGUI1 to K_LEFT1
Connections:
- net COL1: now also K_LGUI1.2 (ROW); no longer K_LGUI1.1 (COL)
- net COL13: now also K_DOWN1.2 (ROW); no longer K_DOWN1.1 (COL)
- net ROW0: now also D37.1 (K)
- net ROW1: now also D43.1 (K)
- net ROW2: now also D48.1 (K)
- net ROW3: now also D53.1 (K)
- net ROW4: now also D58.1 (K)
- net at D74.2 (A): now also K_DOWN1.1 (COL); no longer K_DOWN1.2 (ROW)
- net at D11.2 (A): now also K_LGUI1.1 (COL); no longer K_LGUI1.2 (ROW)
- new net: D37.2 (A), K_EX1.2 (ROW)
- new net: D43.2 (A), K_EX2.2 (ROW)
- new net: D48.2 (A), K_EX3.2 (ROW)
- new net: D53.2 (A), K_EX4.2 (ROW)
- new net: D58.2 (A), K_RIGHT1.2 (ROW)
- new net COL14: K_EX1.1 (COL), K_EX2.1 (COL), K_EX3.1 (COL), K_EX4.1 (COL), K_RIGHT1.1 (COL)
Other:
- moved on the sheet: K_DOWN1, K_LGUI1
Changed lines of the file:
@@
 EESchema Schematic File Version 4
-LIBS:JIS60-cache
+LIBS:JP65-cache
 EELAYER 30 0
 EELAYER END
@@
 	8100 4150 8175 4150
 $Comp
-L MX_Alps_Hybrid:MX-NoLED K_SRSFT2
+L MX_Alps_Hybrid:MX-NoLED K_UP1
 U 1 1 5D497C16
 P 9175 4000
-F 0 "K_SRSFT2" H 9208 4223 60  0000 C CNN
+F 0 "K_UP1" H 9208 4223 60  0000 C CNN
 F 1 "MX-NoLED" H 9208 4149 20  0000 C CNN
-F 2 "MX_Only:MXOnly-1.75U-Hotswap" H 8550 3975 60  0001 C CNN
+F 2 "MX_Only:MXOnly-1U-Hotswap" H 8550 3975 60  0001 C CNN
 F 3 "" H 8550 3975 60  0001 C CNN
 	1    9175 4000
@@
 	6200 4775 6275 4775
 $Comp
-L MX_Alps_Hybrid:MX-NoLED K_RALT1
+L MX_Alps_Hybrid:MX-NoLED K_RCTRL1
 U 1 1 5D497CE6
 P 8225 4625
-F 0 "K_RALT1" H 8258 4848 60  0000 C CNN
+F 0 "K_RCTRL1" H 8258 4848 60  0000 C CNN
 F 1 "MX-NoLED" H 8258 4774 20  0000 C CNN
-F 2 "MX_Only:MXOnly-1U-Hotswap" H 7600 4600 60  0001 C CNN
+F 2 "MX_Only:MXOnly-1.25U-Hotswap" H 7600 4600 60  0001 C CNN
 F 3 "" H 7600 4600 60  0001 C CNN
 	1    8225 4625
@@
 	8100 4775 8175 4775
 $Comp
-L MX_Alps_Hybrid:MX-NoLED K_RCTRL1
+L MX_Alps_Hybrid:MX-NoLED K_DOWN1
 U 1 1 5D497D00
-P 9175 4625
-F 0 "K_RCTRL1" H 9208 4848 60  0000 C CNN
-F 1 "MX-NoLED" H 9208 4774 20  0000 C CNN
-F 2 "MX_Only:MXOnly-1.25U-Hotswap" H 8550 4600 60  0001 C CNN
-F 3 "" H 8550 4600 60  0001 C CNN
-	1    9175 4625
+P 9100 4550
+F 0 "K_DOWN1" H 9133 4773 60  0000 C CNN
+F 1 "MX-NoLED" H 9133 4699 20  0000 C CNN
+F 2 "MX_Only:MXOnly-1U-Hotswap" H 8475 4525 60  0001 C CNN
+F 3 "" H 8475 4525 60  0001 C CNN
+	1    9100 4550
 	1    0    0    -1
 $EndComp
@@
 	0    -1   -1   0
 $EndComp
-Wire Wire Line
-	9050 4775 9125 4775
 Wire Wire Line
 	2875 2475 3350 2475
@@
 Connection ~ 9325 3950
 Wire Wire Line
-	9325 3950 9325 4575
-Wire Wire Line
 	2875 4975 3350 4975
 Wire Wire Line
@@
 L MX_Alps_Hybrid:MX-NoLED K_LGUI1
 U 1 1 5FAA46A7
-P 3475 4625
-F 0 "K_LGUI1" H 3508 4848 60  0000 C CNN
-F 1 "MX-NoLED" H 3508 4774 20  0000 C CNN
-F 2 "MX_Only:MXOnly-1U-Hotswap" H 2850 4600 60  0001 C CNN
-F 3 "" H 2850 4600 60  0001 C CNN
-	1    3475 4625
+P 3400 4550
+F 0 "K_LGUI1" H 3433 4773 60  0000 C CNN
+F 1 "MX-NoLED" H 3433 4699 20  0000 C CNN
+F 2 "MX_Only:MXOnly-1U-Hotswap" H 2775 4525 60  0001 C CNN
+F 3 "" H 2775 4525 60  0001 C CNN
+	1    3400 4550
 	1    0    0    -1
 $EndComp
@@
 	0    -1   -1   0
 $EndComp
-Wire Wire Line
-	3350 4775 3425 4775
 Connection ~ 3350 4975
 Wire Wire Line
@@
 Connection ~ 8850 2075
 $Comp
-L MX_Alps_Hybrid:MX-NoLED K_SRSFT1
+L MX_Alps_Hybrid:MX-NoLED K_RSFT1
 U 1 1 5FB7E4D3
 P 8700 4000
-F 0 "K_SRSFT1" H 8733 4223 60  0000 C CNN
+F 0 "K_RSFT1" H 8733 4223 60  0000 C CNN
 F 1 "MX-NoLED" H 8733 4149 20  0000 C CNN
-F 2 "MX_Only:MXOnly-1U-Hotswap" H 8075 3975 60  0001 C CNN
+F 2 "MX_Only:MXOnly-1.75U-Hotswap" H 8075 3975 60  0001 C CNN
 F 3 "" H 8075 3975 60  0001 C CNN
 	1    8700 4000
@@
 	8575 4350 9050 4350
 $Comp
-L MX_Alps_Hybrid:MX-NoLED K_RGUI1
+L MX_Alps_Hybrid:MX-NoLED K_LEFT1
 U 1 1 5FB9A858
 P 8700 4625
-F 0 "K_RGUI1" H 8733 4848 60  0000 C CNN
+F 0 "K_LEFT1" H 8733 4848 60  0000 C CNN
 F 1 "MX-NoLED" H 8733 4774 20  0000 C CNN
 F 2 "MX_Only:MXOnly-1U-Hotswap" H 8075 4600 60  0001 C CNN
@@
 Connection ~ 8850 3950
 Wire Wire Line
-	3625 3325 3625 4575
-Wire Wire Line
 	2875 4350 3825 4350
 Wire Wire Line
@@
 	0    -1   -1   0
 $EndComp
-Wire Wire Line
-	4300 4775 4375 4775
-Wire Wire Line
-	4575 4575 4575 3950
 Connection ~ 4300 4975
 Wire Wire Line
@@
 	5900 4725 5900 4775
 Connection ~ 6475 4575
+$Comp
+L MX_Alps_Hybrid:MX-NoLED K_EX1
+U 1 1 60F4140F
+P 9650 2125
+F 0 "K_EX1" H 9683 2348 60  0000 C CNN
+F 1 "MX-NoLED" H 9683 2274 20  0000 C CNN
+F 2 "MX_Only:MXOnly-1U-Hotswap" H 9025 2100 60  0001 C CNN
+F 3 "" H 9025 2100 60  0001 C CNN
+	1    9650 2125
+	1    0    0    -1
+$EndComp
+$Comp
+L Device:D_Small D37
+U 1 1 60F41415
+P 9525 2375
+F 0 "D37" V 9571 2307 50  0000 R CNN
+F 1 "SOD-123" V 9480 2307 50  0000 R CNN
+F 2 "Diode_SMD:D_SOD-123" V 9525 2375 50  0001 C CNN
+F 3 "~" V 9525 2375 50  0001 C CNN
+	1    9525 2375
+	0    -1   -1   0
+$EndComp
+Wire Wire Line
+	9525 2275 9600 2275
+$Comp
+L MX_Alps_Hybrid:MX-NoLED K_EX2
+U 1 1 60F4141C
+P 9650 2750
+F 0 "K_EX2" H 9683 2973 60  0000 C CNN
+F 1 "MX-NoLED" H 9683 2899 20  0000 C CNN
+F 2 "MX_Only:MXOnly-1U-Hotswap" H 9025 2725 60  0001 C CNN
+F 3 "" H 9025 2725 60  0001 C CNN
+	1    9650 2750
+	1    0    0    -1
+$EndComp
+$Comp
+L Device:D_Small D43
+U 1 1 60F41422
+P 9525 3000
+F 0 "D43" V 9571 2932 50  0000 R CNN
+F 1 "SOD-123" V 9480 2932 50  0000 R CNN
+F 2 "Diode_SMD:D_SOD-123" V 9525 3000 50  0001 C CNN
+F 3 "~" V 9525 3000 50  0001 C CNN
+	1    9525 3000
+	0    -1   -1   0
+$EndComp
+Wire Wire Line
+	9525 2900 9600 2900
+$Comp
+L MX_Alps_Hybrid:MX-NoLED K_EX3
+U 1 1 60F41429
+P 9650 3375
+F 0 "K_EX3" H 9683 3598 60  0000 C CNN
+F 1 "MX-NoLED" H 9683 3524 20  0000 C CNN
+F 2 "MX_Only:MXOnly-1U-Hotswap" H 9025 3350 60  0001 C CNN
+F 3 "" H 9025 3350 60  0001 C CNN
+	1    9650 3375
+	1    0    0    -1
+$EndComp
+$Comp
+L Device:D_Small D48
+U 1 1 60F4142F
+P 9525 3625
+F 0 "D48" V 9571 3557 50  0000 R CNN
+F 1 "SOD-123" V 9480 3557 50  0000 R CNN
+F 2 "Diode_SMD:D_SOD-123" V 9525 3625 50  0001 C CNN
+F 3 "~" V 9525 3625 50  0001 C CNN
+	1    9525 3625
+	0    -1   -1   0
+$EndComp
+Wire Wire Line
+	9525 3525 9600 3525
+$Comp
+L MX_Alps_Hybrid:MX-NoLED K_EX4
+U 1 1 60F41436
+P 9650 4000
+F 0 "K_EX4" H 9683 4223 60  0000 C CNN
+F 1 "MX-NoLED" H 9683 4149 20  0000 C CNN
+F 2 "MX_Only:MXOnly-1U-Hotswap" H 9025 3975 60  0001 C CNN
+F 3 "" H 9025 3975 60  0001 C CNN
+	1    9650 4000
+	1    0    0    -1
+$EndComp
+$Comp
+L Device:D_Small D53
+U 1 1 60F4143C
+P 9525 4250
+F 0 "D53" V 9571 4182 50  0000 R CNN
+F 1 "SOD-123" V 9480 4182 50  0000 R CNN
+F 2 "Diode_SMD:D_SOD-123" V 9525 4250 50  0001 C CNN
+F 3 "~" V 9525 4250 50  0001 C CNN
+	1    9525 4250
+	0    -1   -1   0
+$EndComp
+Wire Wire Line
+	9525 4150 9600 4150
+$Comp
+L MX_Alps_Hybrid:MX-NoLED K_RIGHT1
+U 1 1 60F41443
+P 9650 4625
+F 0 "K_RIGHT1" H 9683 4848 60  0000 C CNN
+F 1 "MX-NoLED" H 9683 4774 20  0000 C CNN
+F 2 "MX_Only:MXOnly-1U-Hotswap" H 9025 4600 60  0001 C CNN
+F 3 "" H 9025 4600 60  0001 C CNN
+	1    9650 4625
+	1    0    0    -1
+$EndComp
+$Comp
+L Device:D_Small D58
+U 1 1 60F41449
+P 9525 4875
+F 0 "D58" V 9571 4807 50  0000 R CNN
+F 1 "SOD-123" V 9480 4807 50  0000 R CNN
+F 2 "Diode_SMD:D_SOD-123" V 9525 4875 50  0001 C CNN
+F 3 "~" V 9525 4875 50  0001 C CNN
+	1    9525 4875
+	0    -1   -1   0
+$EndComp
+Wire Wire Line
+	9525 4775 9600 4775
+Wire Wire Line
+	9050 2475 9525 2475
+Wire Wire Line
+	9525 3100 9050 3100
+Wire Wire Line
+	9525 3725 9050 3725
+Wire Wire Line
+	9800 2075 9800 2700
+Connection ~ 9800 2700
+Wire Wire Line
+	9800 2700 9800 3325
+Connection ~ 9800 3325
+Text GLabel 9800 1450 0    50   Input ~ 0
+COL14
+Wire Wire Line
+	9800 3325 9800 3950
+Connection ~ 9800 3950
+Wire Wire Line
+	9800 3950 9800 4575
+Connection ~ 9800 2075
+Wire Wire Line
+	9800 1450 9800 2075
+Wire Wire Line
+	9050 4350 9525 4350
+Wire Wire Line
+	9050 4975 9525 4975
+Connection ~ 9050 2475
+Connection ~ 9050 3100
+Connection ~ 9050 3725
+Connection ~ 9050 4350
+Connection ~ 9050 4975
+Wire Wire Line
+	3350 4700 3625 4700
+Wire Wire Line
+	3625 3325 3625 4700
+Wire Wire Line
+	3550 4500 3550 4775
+Wire Wire Line
+	3350 4775 3550 4775
+Wire Wire Line
+	9050 4700 9325 4700
+Wire Wire Line
+	9325 3950 9325 4700
+Wire Wire Line
+	9250 4500 9250 4775
+Wire Wire Line
+	9050 4775 9250 4775
+Wire Wire Line
+	4300 4775 4375 4775
+Wire Wire Line
+	4575 3950 4575 4575
 $EndSCHEMATC
